File: left.kicad_pcb (KiCad board)
At the start: 2 copper layers, 150.9 x 130.2 mm, 80 parts, among them J1 AudioJack4, J2 USB_B_Micro, SW1 SW_DIP_x01, SW10 SW_DIP_x01, SW11 SW_DIP_x01, SW12 SW_DIP_x01, SW13 SW_DIP_x01, SW14 SW_DIP_x01, SW15 SW_DIP_x01, SW16 SW_DIP_x01, SW17 SW_DIP_x01, SW18 SW_DIP_x01, SW19 SW_DIP_x01, SW2 SW_DIP_x01, SW20 SW_DIP_x01, SW21 SW_DIP_x01, SW22 SW_DIP_x01, SW23 SW_DIP_x01, SW24 SW_DIP_x01, SW25 SW_DIP_x01, SW26 SW_DIP_x01, SW27 SW_DIP_x01, SW28 SW_DIP_x01, SW29 SW_DIP_x01, SW3 SW_DIP_x01, SW30 SW_Push_Dual, SW4 SW_DIP_x01, SW5 SW_DIP_x01, SW6 SW_DIP_x01, SW7 SW_DIP_x01, SW8 SW_DIP_x01, SW9 SW_DIP_x01, Y1 16MHz

Commit message: Minor changes.
Parts:
- added REF**: KiCad-Logo2_8mm_SilkScreen, Symbol:KiCad-Logo2_8mm_SilkScreen, F.Cu at (49.7, 14.5)
- added REF**: OSHW-Logo2_14.6x12mm_SilkScreen, Symbol:OSHW-Logo2_14.6x12mm_SilkScreen, F.Cu at (69.2, 15.6)
Other:
- board text added: "Copyright (c) 2021 Herman Lundkvist Grapto Keyboard, Left PCB v1.0"

Commit message: minor changes.
Parts:
- moved C9 171.9 mm to (135.6, 129.7)
- moved D20 171.9 mm to (198.3, 124.3)
- moved D21 171.9 mm to (198.3, 105.2)
- moved D22 171.9 mm to (198.3, 86.1)
- moved D23 171.9 mm to (198.3, 67.0)
- moved SW5 171.9 mm to (137.8, 120.3)
- moved SW6 171.9 mm to (137.8, 101.2)
- moved SW7 171.9 mm to (137.8, 82.1)
- moved SW8 171.9 mm to (137.8, 63.0)
- moved SW9 171.9 mm to (137.8, 43.9)
- moved C1 171.9 mm to (139.3, 150.0)
- moved C10 171.9 mm to (117.4, 134.9)
- moved C11 171.9 mm to (140.2, 142.2)
- moved C12 171.9 mm to (122.4, 128.9)
- moved C13 171.9 mm to (118.0, 141.1)
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